File: PCB Design/Tachometer/Tachometer.kicad_pcb (KiCad board)
At the start: 2 copper layers, 38.1 x 32.2 mm, 52 parts, among them J1 OLED Display Socket, J2 Boot0, J3 USB_B_Micro, J4 UART, J5 SWD, J6 PB_12, J7 PB_13, J8 PB_14, J9 PB_15, SW1 POWER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

Commit message: Fabrications Updated
Parts:
- R4: value 1k -> 500R
- moved D3 61.0 mm to (22.2, 47.1), turned to -90 degrees
- moved SW1 54.9 mm to (46.2, 48.2)
- moved C11 54.6 mm to (28.9, 38.7)
- moved C12 54.6 mm to (28.9, 29.5)
- moved C15 54.6 mm to (40.7, 46.0)
- moved J2 54.6 mm to (48.8, 20.9)
- moved J3 54.6 mm to (52.2, 34.9)
- moved J7 54.6 mm to (48.0, 29.3)
- moved R10 54.6 mm to (28.6, 24.4)
- moved R7 54.6 mm to (48.0, 34.8)
- moved SW4 54.6 mm to (36.1, 48.8)
- moved U1 54.6 mm to (34.0, 41.9)
- moved U2 54.6 mm to (28.1, 44.6)
- moved U3 54.6 mm to (41.4, 32.3)
- moved C3 54.6 mm to (39.6, 24.9)
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Routing:
- net /OP_Out: track 35.0 -> 39.8 mm
- net /VDD: track 169.5 -> 166.5 mm
- net GND: track 8.38 -> 6.37 mm, vias 1 -> 2
- net Net-(D3-K): track 7.40 -> 5.53 mm
- net /Boot0: track 15.8 -> 14.1 mm
- net /Mode_1: track 23.1 -> 24.3 mm
- net /Mode_2: track 25.7 -> 24.8 mm
- net /Reset: track 24.5 -> 25.1 mm
- net /I2C_SCL: track 33.3 -> 32.7 mm
- net Net-(D1-A): track 35.1 -> 34.5 mm
Other:
- board text added: "1"
- board text added: "Off"
- board text added: "Srikar Bharadwaj R RM14"

Commit message: Gerber
Parts:
- moved G*** 0.38 mm to (35.9, 49.0)
- moved G*** 0.38 mm to (35.9, 45.5)
