File: PCB Design/Tachometer/Tachometer-rounded.kicad_pcb (KiCad board)
At the start: 2 copper layers, 38.1 x 32.2 mm, 52 parts, among them J1 OLED Display Socket, J2 Boot0, J3 USB_B_Micro, J4 UART, J5 SWD, J6 PB_12, J7 PB_13, J8 PB_14, J9 PB_15, SW1 POWER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

Commit message: Routed
Routing:
- net GND: track 8.38 -> 2.03 mm
- net /VDD: track 169.5 -> 166.9 mm
- net /VCC: track 57.0 -> 55.4 mm
- net /OP_Out: track 35.0 -> 34.4 mm
- net Net-(D1-A): track 35.1 -> 34.4 mm
- net /HSE_IN: track 11.1 -> 10.5 mm
- net Net-(C12-Pad1): track 7.29 -> 6.78 mm
