File: PCB Design/Tachometer/Tachometer.kicad_sch (KiCad schematic)
At the start: 1 part, among them U1 STM32F405RGT6

Commit message: Schematic
Parts:
- removed U1: STM32F405RGT6, digikey-footprints:LQFP-64_10x10mm, symbol dk_Embedded-Microcontrollers:STM32F405RGT6
- added D1: IR_Receiver, digikey-footprints:LED_5mm_Radial, symbol Device:LED
- added D2: IR_Emitter, digikey-footprints:LED_5mm_Radial, symbol Device:LED
- added D3: Indication LED, digikey-footprints:LED_3mm_Radial, symbol Device:LED
- added J1: OLED Display, Connector_PinSocket_2.54mm:PinSocket_1x07_P2.54mm_Vertical, symbol Connector_Generic:Conn_01x07
- added J2: SWD, Connector_PinHeader_2.54mm:PinHeader_1x04_P2.54mm_Vertical, symbol Connector_Generic:Conn_01x04
- added J3: USB_B_Micro, Connector_USB:USB_Micro-B_GCT_USB3076-30-A, symbol Connector:USB_B_Micro
- added SW1: SW_SPDT, Button_Switch_SMD:SW_SPDT_PCM12, symbol Switch:SW_SPDT
- added U1: LMV321, gsg-modules:SOT25, symbol Amplifier_Operational:LMV321
- added U2: AMS1117, Package_TO_SOT_SMD:SOT-223-3_TabPin2, symbol Regulator_Linear:AMS1117
- added U3: STM32F103C8Tx, Package_QFP:LQFP-48_7x7mm_P0.5mm, symbol MCU_ST_STM32F1:STM32F103C8Tx
- added Y1: Crystal, Crystal:Crystal_HC49-4H_Vertical, symbol Device:Crystal
Connections:
- new net: U3.23 (VSS), U3.35 (VSS), U3.47 (VSS)
- new net CS: J1.7 (Pin_7)
- new net D0: J1.3 (Pin_3)
- new net D1: J1.4 (Pin_4)
- new net DC: J1.6 (Pin_6)
- new net GND: J1.1 (Pin_1)
- new net RES: J1.5 (Pin_5)
- new net Vcc: J1.2 (Pin_2)
Other:
- note added: "Curved Traces"

Commit message: Schematic_Update
Parts:
- removed U2: AMS1117, Package_TO_SOT_SMD:SOT-223-3_TabPin2, symbol Regulator_Linear:AMS1117
- removed Y1: Crystal, Crystal:Crystal_HC49-4H_Vertical, symbol Device:Crystal
- added C1, C11, C2: 10uF, Capacitor_SMD:C_0805_2012Metric_Pad1.18x1.45mm_HandSolder, symbol Device:C
- added C10: 1uF, Capacitor_SMD:C_0805_2012Metric_Pad1.18x1.45mm_HandSolder, symbol Device:C
- added C12, C4, C5, C6, C7, C8, C9: 100nF, Capacitor_SMD:C_0805_2012Metric_Pad1.18x1.45mm_HandSolder, symbol Device:C
- added C13, C3: 24pF, Capacitor_SMD:C_0805_2012Metric_Pad1.18x1.45mm_HandSolder, symbol Device:C
- added FB1: 120R, symbol Device:FerriteBead_Small
- added J4: UART, Connector_PinHeader_2.54mm:PinHeader_1x04_P2.54mm_Vertical, symbol Connector_Generic:Conn_01x04
- added J5: Boot0, Connector_PinHeader_1.27mm:PinHeader_1x03_P1.27mm_Vertical_SMD_Pin1Left, symbol Connector:Conn_01x03_Pin
- added R1: 0R, Resistor_SMD:R_0603_1608Metric_Pad0.98x0.95mm_HandSolder, symbol Device:R_US
- added R2, R4, R6: 10k, Resistor_SMD:R_0603_1608Metric_Pad0.98x0.95mm_HandSolder, symbol Device:R_US
- added R3: 1k, Resistor_SMD:R_0603_1608Metric_Pad0.98x0.95mm_HandSolder, symbol Device:R_US
- added R5: 100R, Resistor_SMD:R_1206_3216Metric_Pad1.30x1.75mm_HandSolder, symbol Device:R_US
- added R7, R8, R9: 1.5k, Resistor_SMD:R_0603_1608Metric_Pad0.98x0.95mm_HandSolder, symbol Device:R_US
- added RV1: 10k, Potentiometer_THT:Potentiometer_Bourns_3296Y_Vertical, symbol Device:R_Potentiometer_Trim
- added SW2: Reset, symbol Switch:SW_Push
- added U4: AMS1117-3.3, Package_TO_SOT_SMD:SOT-223-3_TabPin2, symbol Regulator_Linear:AMS1117-3.3
- added Y2: ABM3B-8.000MHZ-B2-T, symbol Device:Crystal_GND24_Small
- D3: footprint digikey-footprints:LED_3mm_Radial -> LED_SMD:LED_0603_1608Metric_Pad1.05x0.95mm_HandSolder
Connections:
- net GND: now also J2.4 (Pin_4), J3.5 (GND), U1.2 (V-), U3.23 (VSS), U3.35 (VSS), U3.47 (VSS), U3.8 (VSSA), C1.2, C10.2, C11.2, C12.2, C13.2, C2.2, C3.2, C4.2, C5.2, C6.2, C7.2, C8.2, C9.2, J4.4 (Pin_4), J5.3 (Pin_3), R2.2, R3.2, R4.2, R5.2, RV1.3, SW2.1, U4.1 (GND), Y2.2, Y2.4
- net VDD: now reaches J2.1 (Pin_1)
- net VDD: now also U3.1 (VBAT), U3.24 (VDD), U3.36 (VDD), U3.48 (VDD), C11.1, C2.1, C4.1, C5.1, C6.1, C7.1, C9.1, FB1.2, J4.1 (Pin_1), J5.1 (Pin_1), R7.2, R8.2, R9.2, U4.2 (VO)
- net SWDIO: now reaches J2.2 (Pin_2)
- net SWDIO: now also U3.34 (PA13)
- net SWCLK: now reaches J2.3 (Pin_3)
- net SWCLK: now also U3.37 (PA14)
- net VCC: now reaches D1.1 (K)
- net VCC: now also D2.2 (A), SW1.1 (A), U1.5 (V+), C1.1, RV1.1, U4.3 (VI)
- net at D1.2 (A): now also U1.1 (+), R4.1
- net VBUS: now reaches J3.1 (VBUS)
- net VBUS: now also SW1.2 (B)
- net USB_D-: now reaches J3.2 (D-)
- net USB_D-: now also U3.32 (PA11)
- net USB_D+: now reaches J3.3 (D+)
- net USB_D+: now also U3.33 (PA12), R7.1
- net at D2.1 (K): now also R5.1
- net at U1.3 (-): now also RV1.2
- net OP_Out: now reaches U1.4
- net OP_Out: now also D3.2 (A), U3.46 (PB9), R2.1
- net at D3.1 (K): now also R3.1
- net UART_Tx: now reaches U3.12 (PA2)
- net UART_Tx: now also J4.2 (Pin_2)
- net UART_Rx: now reaches U3.13 (PA3)
- net UART_Rx: now also J4.3 (Pin_3)
- net I2C_SCL: now reaches U3.42 (PB6)
- net I2C_SCL: now also R8.1
- net I2C_SDA: now reaches U3.43 (PB7)
- net I2C_SDA: now also R9.1
- net Boot0: now reaches U3.44 (BOOT0)
- net Boot0: now also R6.2
- net HSE_IN: now reaches U3.5 (PD0)
- net HSE_IN: now also C3.1, Y2.1
- net HSE_OUT: now reaches U3.6 (PD1)
- net HSE_OUT: now also R1.2
- net at U3.7 (NRST): now also C12.1, SW2.2
- net VDDA: now reaches U3.9 (VDDA)
- net VDDA: now also C10.1, C8.1, FB1.1
- new net: C13.1, R1.1, Y2.3
- new net: J5.2 (Pin_2), R6.1
- no-connect marks 0 -> 3
Other:
- note added: "GitHub Link"
- note added: "IR Sensor Circuit"
- note added: "Micro Controller Unit"
- note added: "Peripherals"
- note added: "Power Circuit"
- note added: "USB Circuit"
- company: (none) -> RoboManipal
- title: (none) -> Project Tachometer
- moved on the sheet: D1, D2, D3, J1, J2, J3, SW1, U1, U3

Commit message: PCB_Routed
Parts:
- removed J1: OLED Display, Connector_PinSocket_2.54mm:PinSocket_1x07_P2.54mm_Vertical, symbol Connector_Generic:Conn_01x07
- removed Y2: ABM3B-8.000MHZ-B2-T, symbol Device:Crystal_GND24_Small
- added C14, C15: 1uF, Capacitor_SMD:C_0805_2012Metric_Pad1.18x1.45mm_HandSolder, symbol Device:C
- added J1: OLED Display Socket, Connector_PinSocket_2.54mm:PinSocket_1x04_P2.54mm_Vertical, symbol Connector_Generic:Conn_01x04
- added J2: OLED Display, SSD1306:128x64OLED, symbol Connector_Generic:Conn_01x04
- added R10, R11, R12: 10k, Resistor_SMD:R_0603_1608Metric_Pad0.98x0.95mm_HandSolder, symbol Device:R_US
- added SW3: Mode_1, Button_Switch_SMD:SW_TS09-63-25-WT-160-SMT-TR, symbol Switch:SW_Push
- added SW4: Mode_2, Button_Switch_SMD:SW_TS09-63-25-WT-160-SMT-TR, symbol Switch:SW_Push
- added Y1: 8MHz_Crystal, Crystal:Crystal_SMD_HC49-SD, symbol Device:Crystal
- C11: renamed from C3; value 24pF -> 33pF
- C12: renamed from C13; value 24pF -> 33pF
- C13: renamed from C12; value 100nF -> 1uF
- FB1: footprint (none) -> Inductor_SMD:L_0603_1608Metric_Pad1.05x0.95mm_HandSolder
- J3: renamed from J5; footprint Connector_PinHeader_1.27mm:PinHeader_1x03_P1.27mm_Vertical_SMD_Pin1Left -> Connector_PinHeader_2.54mm:PinHeader_1x03_P2.54mm_Vertical
- R5: footprint Resistor_SMD:R_1206_3216Metric_Pad1.30x1.75mm_HandSolder -> Resistor_THT:R_Axial_DIN0204_L3.6mm_D1.6mm_P5.08mm_Horizontal
- RV1: footprint Potentiometer_THT:Potentiometer_Bourns_3296Y_Vertical -> Potentiometer_THT:Potentiometer_Bourns_3296W_Vertical
- SW2: footprint (none) -> Button_Switch_SMD:SW_TS09-63-25-WT-160-SMT-TR
- renumbered C7 to C10, C8 to C3, C10 to C4, C9 to C5, C11 to C6, C4 to C7, C5 to C8, C6 to C9, J3 to J4, J4 to J5, J2 to J6, R6 to R1, R4 to R2, R2 to R3, R3 to R4, R1 to R6, U4 to U1, U1 to U2
Connections:
- net GND: now also C13.1, SW2.2, J1.1 (Pin_1), J2.1 (Pin_1), R11.1, R12.1; no longer C13.2, SW2.1
- net HSE_IN: now also Y1.1
- net I2C_SCL: now also J1.3 (Pin_3), J2.3 (Pin_3)
- net I2C_SDA: now also J1.4 (Pin_4), J2.4 (Pin_4)
- net OP_Out: now also U3.38 (PA15); no longer U3.46 (PB9)
- net UART_Rx: now also U3.31 (PA10); no longer U3.13 (PA3)
- net UART_Tx: now also U3.30 (PA9); no longer U3.12 (PA2)
- net VDD: now also C14.2, C15.2, J1.2 (Pin_2), J2.2 (Pin_2), R10.2, SW3.1, SW4.1
- net at C12.1, R6.1: now also Y1.2
- net Mode_1: now reaches U3.39 (PB3)
- net Mode_1: now also C14.1, R11.2, SW3.2
- net Mode_2: now reaches U3.40 (PB4)
- net Mode_2: now also C15.1, R12.2, SW4.2
- new net Reset: C13.2, R10.1, SW2.1, U3.7 (NRST)
- no-connect marks 3 -> 27
Other:
- note added: "Add Solder Plates if possible for GPIOs"
- note added: "CLoad = 20pF, => C1 = C2 = 2*(20-4), assuming C_stray = 4pF"
- note added: "Crystal Link"
- note added: "Open Source Hardware"
- note added: "Skeptical about this"
- note removed: "USB Circuit"
- moved on the sheet: C10, C11, C12, C13, C3, C4, C5, C6, C7, C8, C9, FB1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

Commit message: Routed
Parts:
- removed J2: OLED Display, SSD1306:128x64OLED, symbol Connector_Generic:Conn_01x04
- added J6: PB_12, Connector_Wire:SolderWirePad_1x01_SMD_1x2mm, symbol Connector:Conn_01x01_Pin
- added J7: PB_13, Connector_Wire:SolderWirePad_1x01_SMD_1x2mm, symbol Connector:Conn_01x01_Pin
- added J8: PB_14, Connector_Wire:SolderWirePad_1x01_SMD_1x2mm, symbol Connector:Conn_01x01_Pin
- added J9: PB_15, Connector_Wire:SolderWirePad_1x01_SMD_1x2mm, symbol Connector:Conn_01x01_Pin
- SW1: value SW_SPDT -> POWER
- renumbered J3 to J2, J4 to J3, J5 to J4, J6 to J5
Connections:
- net GND: now also RV1.1; no longer RV1.3
- net VCC: now also RV1.3; no longer RV1.1
- net at U3.25 (PB12): now also J6.1 (Pin_1)
- net at U3.26 (PB13): now also J7.1 (Pin_1)
- net at U3.27 (PB14): now also J8.1 (Pin_1)
- net at U3.28 (PB15): now also J9.1 (Pin_1)
- no-connect marks 27 -> 23
Other:
- note removed: "Add Solder Plates if possible for GPIOs"
- note removed: "Curved Traces"

Commit message: Fabrications Updated
Parts:
- R4: value 1k -> 500R
